File: schematics/diagnostics/diagnostics.kicad_sch (KiCad schematic)
At the start: 10 parts, among them J2 Conn_01x06_Socket, J3 Conn_02x04_Odd_Even

Commit message: Signed-off-by: Ray33ee <30669752+ray33ee@users.noreply.github.com>
Parts:
- added C1: 0.1uF, Capacitor_SMD:C_1206_3216Metric_Pad1.33x1.80mm_HandSolder, symbol Device:C
- added J1: USB_B_Micro, symbol Connector:USB_B_Micro
- added U1: CH340N, Package_SO:SOP-8_3.9x4.9mm_P1.27mm, symbol Interface_USB:CH340N
Connections:
- net +3V3: now also C1.1, U1.5 (VCC), U1.8 (V3)
- net GND: now also C1.2, J1.5 (GND), J1.6 (Shield), U1.3 (GND)
- net RX: now also U1.7 (RXD)
- net TX: now also U1.6 (TXD)
- new net D+: J1.3 (D+), U1.1 (UD+)
- new net D-: J1.2 (D-), U1.2 (UD-)
- no-connect marks 4 -> 7
Other:
- moved on the sheet: D1, D2, D3, D4, J2, J3, R1, R2, R3, R4

Commit message: Signed-off-by: Ray33ee <30669752+ray33ee@users.noreply.github.com>
Parts:
- removed J1: USB_B_Micro, symbol Connector:USB_B_Micro
- removed J2: Conn_01x06_Socket, Connector_PinSocket_2.54mm:PinSocket_1x06_P2.54mm_Horizontal, symbol Connector:Conn_01x06_Socket
- removed J3: Conn_02x04_Odd_Even, Connector_PinHeader_2.54mm:PinHeader_2x04_P2.54mm_Horizontal, symbol Connector_Generic:Conn_02x04_Odd_Even
- added J1: SAMTEC-MMT-104-02-X-DH, custom:SAMTEC-MMT-104-02-X-DH, symbol custom:SAMTEC-MMT-104-02-X-DH
- added R5, R6: 0603WAF5101T5E, Resistor_SMD:R_0603_1608Metric, symbol Device:R
- added USB1: TYPE-C-31-M-13, custom:USB-C-SMD_TYPE-C-31-M-13, symbol custom:TYPE-C-31-M-13
Connections:
- net +3V3: now also J1.7
- net D+: now also USB1.A6 (DP1), USB1.B6 (DP2)
- net D-: now also USB1.A7 (DN1), USB1.B7 (DN2)
- net EXCEPTION: now also J1.5
- net GND: now also J1.8, R5.1, R6.2, USB1.0 (EP), USB1.A1 (GND), USB1.A12 (GND), USB1.B1 (GND), USB1.B12 (GND)
- net HEART: now also J1.1
- net PANIC: now also J1.3
- net RX: now also J1.2
- net TX: now also J1.6
- net PWR: now reaches D4.1 (K), R4.2
- net EXC: now reaches D1.1 (K), R1.2
- net BEAT: now reaches D3.1 (K), R3.2
- net PAN: now reaches D2.1 (K), R2.2
- new net: R6.1, USB1.A5 (CC1)
- new net: R5.2, USB1.B5 (CC2)
- no-connect marks 7 -> 8
Other:
- moved on the sheet: C1, D1, D2, D3, D4, R1, R2, R3, R4, U1
