File: schematics/top/top.kicad_pcb (KiCad board)
At the start: 2 copper layers, 45.1 x 45.1 mm, 13 parts, among them J1 CLT-108-02-F-D-BE-K-TR, J2 Conn_01x04_Socket

Commit message: Signed-off-by: Ray33ee <30669752+ray33ee@users.noreply.github.com>
Parts:
- removed ? (x2): , 
- removed REF**: MountingHole_4mm, MountingHole:MountingHole_4mm
- JP1: moved to B.Cu
- moved JP2 23.5 mm to (143.4, 116.5)
- moved JP1 14.7 mm to (133.1, 116.5)
- moved JP3 11.2 mm to (137.7, 113.3), turned to 90 degrees
- moved U1 0.06 mm to (120.1, 105.2), turned to 90 degrees
Routing:
- net GND: track 0.00 -> 58.4 mm, vias 0 -> 2
- net /SDA: track 7.20 -> 32.1 mm
- net /SCL: track 4.07 -> 23.7 mm, vias 0 -> 1
- net +3V3: track 55.4 -> 65.6 mm, vias 0 -> 2
- net DATA2: track 31.8 -> 27.7 mm, vias 2 -> 0
- net DATA1: track 33.6 -> 36.6 mm, vias 2 -> 1
- net /G: track 18.8 -> 16.8 mm
- net /1WIRE: track 8.95 -> 8.71 mm, vias 2 -> 0
- removed copper zone on F.Cu, net GND
Other:
- board size 45.1 x 45.1 mm -> 44.9 x 45.1 mm

Commit message: Signed-off-by: Ray33ee <30669752+ray33ee@users.noreply.github.com>
Parts:
- added JP4: SolderJumper_2_Open, Jumper:SolderJumper-2_P1.3mm_Open_RoundedPad1.0x1.5mm, F.Cu at (143.4, 112.3)
- U1: value ~ -> AHT20-F
Connections:
- net /1WIRE renamed /D1
- J2 pad 2: unconnected-(J2-Pin_2-Pad2) -> /D2
Routing:
- net /D2: track 0.00 -> 15.0 mm, vias 0 -> 2
- net DATA2: track 27.7 -> 35.6 mm, vias 0 -> 2

Commit message: Signed-off-by: Ray33ee <30669752+ray33ee@users.noreply.github.com>
Other:
- board text added: "v0.1.0"
Changed lines of the file:
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@@
 		(attr smd)
 		(fp_line
-			(start -2.1 -1.15)
-			(end -1.6 -1.65)
+			(start -2.1 -1.2)
+			(end -1.6 -1.7)
 			(stroke
 				(width 0.12)
@@
 		)
 		(pad "1" smd rect
-			(at -1.25 -0.7)
+			(at -1.75 -0.7)
 			(size 1.6 0.8)
 			(layers "F.Cu" "F.Mask" "F.Paste")
@@
 		)
 		(pad "2" smd rect
-			(at -1.25 0.7)
+			(at -1.75 0.7)
 			(size 1.6 0.8)
 			(layers "F.Cu" "F.Mask" "F.Paste")
@@
 		)
 		(pad "3" smd rect
-			(at 1.25 0.7)
+			(at 1.75 0.7)
 			(size 1.6 0.8)
 			(layers "F.Cu" "F.Mask" "F.Paste")
@@
 		)
 		(pad "4" smd rect
-			(at 1.25 -0.7)
+			(at 1.75 -0.7)
 			(size 1.6 0.8)
 			(layers "F.Cu" "F.Mask" "F.Paste")
@@
 	(gr_rect
 		(start 123.22 113.28)
+		(end 126.22 115.78)
+		(stroke
+			(width 0.2)
+			(type solid)
+		)
+		(fill yes)
+		(layer "F.Mask")
+	)
+	(gr_rect
+		(start 123.22 116.78)
 		(end 126.22 119.28)
 		(stroke
@@
 		(layer "User.2")
 	)
+	(gr_text "v0.1.0"
+		(at 131.22 87.28 -0)
+		(layer "B.SilkS")
+		(effects
+			(font
+				(size 1 1)
+				(thickness 0.15)
+			)
+			(justify left bottom mirror)
+		)
+	)
 	(segment
 		(start 144.271 99.130074)
@@
 	)
 	(segment
-		(start 133.42 101.51)
+		(start 133.42 102.012)
 		(end 133.42 99.88)
 		(width 0.2)
@@
 	)
 	(segment
-		(start 136.85 104.54)
-		(end 136.45 104.54)
+		(start 135.948 104.54)
+		(end 133.42 102.012)
+		(width 0.2)
+		(layer "F.Cu")
+		(net 20)
+	)
+	(segment
+		(start 133.42 99.88)
+		(end 140.22 93.08)
 		(width 0.2)
 		(layer "F.Cu")
@@
 	)
 	(segment
-		(start 136.45 104.54)
-		(end 133.42 101.51)
+		(start 136.85 104.54)
+		(end 136.45 104.54)
 		(width 0.2)
 		(layer "F.Cu")
@@
 	)
 	(segment
-		(start 133.42 99.88)
-		(end 140.22 93.08)
+		(start 136.35 104.54)
+		(end 135.948 104.54)
 		(width 0.2)
 		(layer "F.Cu")
@@
 	)
 	(segment
-		(start 139.42 104.61)
-		(end 139.35 104.54)
-		(width 0.2)
-		(layer "F.Cu")
-		(net 22)
-	)
-	(segment
