File: schematics/front/front.kicad_pcb (KiCad board)
At the start: 2 copper layers, 29.1 x 46.8 mm, 28 parts, among them J1 USB_B_Micro, J2 MOTOR, J4 RGB, J5 THERMO, SW1 RESET, SW2 BOOT, SW3 MODE, U1 ME6211C33M5, U2 ESP32-S2-MINI-2-N4, U3 DRV8836

Commit message: Signed-off-by: Ray33ee <30669752+ray33ee@users.noreply.github.com>
Parts:
- removed D1: XL-1615RGBC-RF, Resistor_SMD:R_Array_Convex_2x0606
- removed J4: RGB, Connector_JST:JST_SH_SM04B-SRSS-TB_1x04-1MP_P1.00mm_Horizontal
- removed J5: THERMO, Connector_JST:JST_SH_SM04B-SRSS-TB_1x04-1MP_P1.00mm_Horizontal
- removed R10, R8, R9: 10k, Resistor_SMD:R_0603_1608Metric
- removed R6, R7: R, Resistor_SMD:R_1206_3216Metric
- added J3: Conn_01x08_Pin, connector:SAMTEC-MMT-108-02-X-SH, F.Cu at (138.3, 69.8)
- added J6: Conn_02x04_Odd_Even, connector:SAMTEC_CLT-104-02-F-D-BE-K-TR, F.Cu at (143.4, 84.8)
- added JP1: SolderJumper_2_Bridged, Jumper:SolderJumper-2_P1.3mm_Bridged_RoundedPad1.0x1.5mm, B.Cu at (127.8, 80.8)
- added JP2: SolderJumper_2_Bridged, Jumper:SolderJumper-2_P1.3mm_Bridged_RoundedPad1.0x1.5mm, B.Cu at (131.4, 80.8)
- added JP3: SolderJumper_2_Open, Jumper:SolderJumper-2_P1.3mm_Open_RoundedPad1.0x1.5mm, B.Cu at (135.6, 93.3)
- added JP4: SolderJumper_2_Open, Jumper:SolderJumper-2_P1.3mm_Open_RoundedPad1.0x1.5mm, B.Cu at (131.7, 94.9)
- added JP5: SolderJumper_2_Open, Jumper:SolderJumper-2_P1.3mm_Open_RoundedPad1.0x1.5mm, B.Cu at (136.6, 78.3)
- added JP6: SolderJumper_2_Open, Jumper:SolderJumper-2_P1.3mm_Open_RoundedPad1.0x1.5mm, B.Cu at (136.6, 83.1)
- added R11: 0603WAF3302T5E, Resistor_SMD:R_0603_1608Metric, F.Cu at (135.6, 81.7)
- added R12: 0603WAF3302T5E, Resistor_SMD:R_0603_1608Metric, F.Cu at (135.6, 80.0)
- added R13: 0603WAF6802T5E, Resistor_SMD:R_0603_1608Metric, F.Cu at (135.6, 78.3)
- added R14: 0603WAF6802T5E, Resistor_SMD:R_0603_1608Metric, F.Cu at (135.7, 83.4)
- added R15: 0603WAF6802T5E, Resistor_SMD:R_0603_1608Metric, F.Cu at (124.4, 78.5)
- added R16: 0603WAF3302T5E, Resistor_SMD:R_0603_1608Metric, F.Cu at (124.4, 80.1)
- added R17: 0603WAF6802T5E, Resistor_SMD:R_0603_1608Metric, F.Cu at (124.4, 83.3)
- added R18: 0603WAF3302T5E, Resistor_SMD:R_0603_1608Metric, F.Cu at (124.4, 81.7)
- J2: moved to B.Cu
- R1, R2: value 5.1k -> 1; footprint Resistor_SMD:R_0603_1608Metric -> Resistor_SMD:R_1206_3216Metric_Pad1.30x1.75mm_HandSolder
- R3: value 10k -> 0603WAF1002T5E
- R4: value 10k -> 0603WAF1002T5E; footprint Resistor_SMD:R_1206_3216Metric -> Resistor_SMD:R_0603_1608Metric
- R5: value R -> 0603WAF1002T5E; footprint Resistor_SMD:R_1206_3216Metric -> Resistor_SMD:R_0603_1608Metric
- U1: value ME6211C33M5 -> LD1117AG-33-AA3-A-R; footprint Package_TO_SOT_SMD:SOT-23-5 -> Package_TO_SOT_SMD:SOT-223-3_TabPin2
- moved C1 34.4 mm to (148.8, 118.3), turned to 180 degrees
- moved U1 32.1 mm to (146.5, 113.0), turned to 90 degrees
- moved C2 31.8 mm to (145.7, 118.3), turned to 180 degrees
- moved R5 31.4 mm to (143.0, 79.5), turned to 180 degrees
- moved C3 29.7 mm to (130.8, 111.2), turned to 0 degrees
- moved C5 29.4 mm to (128.2, 112.0), turned to -90 degrees
- moved SW1 29.1 mm to (146.8, 105.5), turned to 0 degrees
- moved C4 27.9 mm to (130.8, 113.1), turned to 0 degrees
- moved C6 22.8 mm to (148.8, 102.2)
- moved SW3 22.1 mm to (126.6, 116.7), turned to 180 degrees
- moved R3 17.7 mm to (147.2, 101.2), turned to -90 degrees
- moved R2 16.1 mm to (128.1, 80.9), turned to -90 degrees
- moved R4 12.0 mm to (143.0, 77.7), turned to 180 degrees
- moved R1 10.1 mm to (131.2, 80.9), turned to -90 degrees
- moved U3 6.43 mm to (132.0, 89.1)
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Connections:
- net Net-(J2-Pin_1) renamed A1
- J2 pad 2: Net-(J2-Pin_2) -> B1
- J2 pad 3: Net-(J2-Pin_3) -> /_A2
- R1 pad 1: Net-(USB1-CC2) -> /_A2
- R1 pad 2: GND -> A2
- R2 pad 1: Net-(USB1-CC1) -> Net-(J2-Pin_4)
- R2 pad 2: GND -> B2
- R4 pad 1: IO18 -> +3V3
- R4 pad 2: +3V3 -> DATA2
- R5 pad 1: RED1 -> +3V3
- R5 pad 2: Net-(D1-RK) -> DATA1
- U1 pad 1: VBUS -> GND
- U1 pad 2: GND -> +3V3
- U2 pad 10: unconnected-(U2-IO6-Pad10) -> SENSE2
- U2 pad 11: unconnected-(U2-IO7-Pad11) -> SENSE1
- U2 pad 17: unconnected-(U2-IO13-Pad17) -> DATA2
- U2 pad 18: unconnected-(U2-IO14-Pad18) -> DATA1
- U2 pad 19: unconnected-(U2-IO15-Pad19) -> BLUE
- U2 pad 20: unconnected-(U2-IO16-Pad20) -> GREEN
- U2 pad 21: unconnected-(U2-IO17-Pad21) -> RED
- U2 pad 22: IO18 -> unconnected-(U2-IO18-Pad22)
- U2 pad 25: unconnected-(U2-IO21-Pad25) -> EXCEPTION
- U2 pad 26: unconnected-(U2-IO26-Pad26) -> PANIC
- U2 pad 28: unconnected-(U2-IO33-Pad28) -> HEART
- U2 pad 31: unconnected-(U2-IO35-Pad31) -> RX
- U2 pad 32: unconnected-(U2-IO36-Pad32) -> TX
- U2 pad 35: unconnected-(U2-IO39-Pad35) -> nSLEEP
- U2 pad 36: unconnected-(U2-IO40-Pad36) -> AIN1
- U2 pad 37: unconnected-(U2-IO41-Pad37) -> AIN2
- U2 pad 38: unconnected-(U2-IO42-Pad38) -> BIN1
- U2 pad 41: unconnected-(U2-IO45-Pad41) -> BIN2
- U2 pad 7: unconnected-(U2-IO3-Pad7) -> MODE
- U2 pad 8: unconnected-(U2-IO4-Pad8) -> SENSE3
- U2 pad 9: unconnected-(U2-IO5-Pad9) -> SENSE4
- U3 pad 3: Net-(J2-Pin_2) -> A2
- U3 pad 4: Net-(J2-Pin_3) -> B1
- U3 pad 5: Net-(J2-Pin_4) -> B2
Routing:
- net +3V3: track 0.00 -> 91.3 mm, vias 0 -> 9
- net VBUS: track 0.00 -> 61.6 mm, vias 0 -> 2
- net DATA1: track 0.00 -> 53.1 mm, vias 0 -> 2
- net DATA2: track 0.00 -> 51.1 mm, vias 0 -> 2
- net BLUE: track 0.00 -> 47.9 mm, vias 0 -> 2
- net SENSE3: track 0.00 -> 43.9 mm, vias 0 -> 1
- net GREEN: track 0.00 -> 41.3 mm, vias 0 -> 2
- net RED: track 0.00 -> 37.5 mm, vias 0 -> 2
- net SENSE4: track 0.00 -> 37.0 mm, vias 0 -> 1
- net EN: track 0.00 -> 34.0 mm, vias 0 -> 3
- net IO0: track 0.00 -> 32.1 mm, vias 0 -> 2
- net D-: track 0.00 -> 27.6 mm, vias 0 -> 1
- net D+: track 0.00 -> 27.3 mm, vias 0 -> 1
- net EXCEPTION: track 0.00 -> 26.5 mm, vias 0 -> 2
- net SENSE1: track 0.00 -> 26.0 mm, vias 0 -> 1
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- added copper zone on In1.Cu, net GND
- added copper zone on In2.Cu, net GND
Other:
- board size 29.1 x 46.8 mm -> 29.1 x 51.8 mm
- copper layers 2 -> 4
- board text added: "BOOT"
- board text added: "MODE"
- board text added: "RESET"

Commit message: Signed-off-by: Ray33ee <30669752+ray33ee@users.noreply.github.com>
Connections:
- J6 pad 1: EXCEPTION -> HEART
- J6 pad 5: HEART -> EXCEPTION
- U2 pad 25: EXCEPTION -> HEART
- U2 pad 28: HEART -> EXCEPTION
Routing:
- net HEART: track 18.9 -> 26.5 mm
- net EXCEPTION: track 26.5 -> 18.9 mm
- net GND: vias 516 -> 678

Commit message: Signed-off-by: Ray33ee <30669752+ray33ee@users.noreply.github.com>
Changed lines of the file:
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@@
 		(allow_soldermask_bridges_in_footprints no)
 		(tenting front back)
-		(grid_origin 131.05 99)
+		(grid_origin 134.25 87.375)
 		(pcbplotparams
 			(layerselection 0x00000000_00000000_55555555_5755f5ff)
@@
 		(tags "resistor")
 		(property "Reference" "R14"
-			(at -2.875 0.05 0)
+			(at -2.875 0 0)
 			(layer "F.SilkS")
 			(effects
@@
 		(embedded_fonts no)
 	)
+	(gr_rect
+		(start 133.95 86.975)
+		(end 138.05 91.675)
+		(stroke
+			(width 0.1)
+			(type solid)
+		)
+		(fill yes)
+		(layer "F.Mask")
+	)
+	(gr_rect
+		(start 128.15 85.175)
+		(end 130.05 91.075)
+		(stroke
+			(width 0.1)
+			(type solid)
+		)
+		(fill yes)
+		(layer "F.Mask")
+	)
 	(gr_line

Commit message: Signed-off-by: Ray33ee <30669752+ray33ee@users.noreply.github.com>
Parts:
- removed JP1, JP2: SolderJumper_2_Bridged, Jumper:SolderJumper-2_P1.3mm_Bridged_RoundedPad1.0x1.5mm
- removed JP3, JP4, JP5, JP6: SolderJumper_2_Open, Jumper:SolderJumper-2_P1.3mm_Open_RoundedPad1.0x1.5mm
- removed R1, R2: 1, Resistor_SMD:R_1206_3216Metric_Pad1.30x1.75mm_HandSolder
- removed R11, R12, R16, R18: 0603WAF3302T5E, Resistor_SMD:R_0603_1608Metric
- removed R13, R14, R15, R17: 0603WAF6802T5E, Resistor_SMD:R_0603_1608Metric
- moved J2 13.2 mm to (141.2, 74.7)
- moved SW3 2.76 mm to (129.3, 116.5), turned to -90 degrees
- moved U2 0.50 mm to (134.8, 102.2)
- moved C4 0.32 mm to (130.8, 112.8)
- moved C5 0.20 mm to (128.4, 112.0)
Connections:
- J2 pad 3: /_A2 -> A2
- J2 pad 4: Net-(J2-Pin_4) -> B2
- U2 pad 10: SENSE2 -> unconnected-(U2-IO6-Pad10)
- U2 pad 11: SENSE1 -> unconnected-(U2-IO7-Pad11)
- U2 pad 26: PANIC -> unconnected-(U2-IO26-Pad26)
- U2 pad 28: EXCEPTION -> PANIC
- U2 pad 29: unconnected-(U2-IO34-Pad29) -> EXCEPTION
- U2 pad 8: SENSE3 -> unconnected-(U2-IO4-Pad8)
- U2 pad 9: SENSE4 -> unconnected-(U2-IO5-Pad9)
Routing:
- net SENSE3: track 43.9 -> 0.00 mm, vias 1 -> 0
- net SENSE4: track 37.0 -> 0.00 mm, vias 1 -> 0
- net SENSE1: track 26.0 -> 0.00 mm, vias 1 -> 0
- net SENSE2: track 25.3 -> 0.00 mm, vias 1 -> 0
- net /S1: track 22.2 -> 0.00 mm, vias 1 -> 0
- net /S2: track 21.7 -> 0.00 mm, vias 1 -> 0
- net A2: track 11.8 -> 28.1 mm, vias 2 -> 1
- net /_A2: track 14.2 -> 0.00 mm, vias 2 -> 0
- net B2: track 13.0 -> 26.9 mm, vias 2 -> 1
- net Net-(J2-Pin_4): track 12.3 -> 0.00 mm, vias 3 -> 0
- net A1: track 17.1 -> 27.9 mm
- net B1: track 17.1 -> 27.7 mm
- net DATA1: track 53.1 -> 48.3 mm
- net /S4: track 4.32 -> 0.00 mm, vias 1 -> 0
- net /S3: track 4.32 -> 0.00 mm, vias 1 -> 0
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
Commit message: Signed-off-by: Ray33ee <30669752+ray33ee@users.noreply.github.com>
Parts:
- added ?: , , F.Cu at (148.9, 70.5)
- added REF**: MountingHole_2.1mm, MountingHole:MountingHole_2.1mm, F.Cu at (123.0, 119.3)
- moved J4 2.00 mm to (141.4, 84.8)
- moved C2 1.21 mm to (144.5, 118.2)
- moved C1 0.76 mm to (148.0, 118.2)
- moved J2 0.50 mm to (140.7, 74.7)
- moved J3 0.50 mm to (137.8, 69.8)
- moved R2 0.10 mm to (143.0, 79.4)
- renumbered J6 to J4, R3 to R1, R5 to R2, R4 to R3
Connections:
- net A1 renamed A1(WHITE)
- net A2 renamed A2(BLACK)
- net B1 renamed B1(YELLOW)
- net B2 renamed B2(RED)
Routing:
- net +3V3: track 91.8 -> 94.7 mm
- net PANIC: track 21.7 -> 23.7 mm
- net HEART: track 26.0 -> 28.0 mm
- net EXCEPTION: track 18.0 -> 20.0 mm
- net GREEN: track 40.8 -> 41.5 mm
- net RX: track 10.1 -> 10.7 mm
- net A2(BLACK): track 28.1 -> 27.6 mm
- net GND: vias 757 -> 797
Other:
- board size 29.1 x 51.8 mm -> 28.9 x 51.8 mm
- board text added: "V0.1.0"
